File: Schematic/Analog_AFE.sch (KiCad schematic (older format))
At the start: 49 parts, among them IC1 ADS1299-4PAGR

Commit message: Add files via upload
Parts:
- added R235, R236: R_Small, Resistor_SMD:R_0402_1005Metric, symbol Device:R_Small
Connections:
- net GNDD is gone; now on net GND: C29.1, C31.2, IC1.33 (DGND_1), IC1.41 (DAISY_IN), IC1.49 (DGND_2), IC1.51 (DGND_3)
- net nPWDN: now also R236.1; no longer IC1.35 (~PWDN)
- net nRESET: now also R235.1; no longer IC1.36 (~RESET)
- net GNDA renamed GND
- new net: IC1.35 (~PWDN), R236.2
- new net: IC1.36 (~RESET), R235.2
Changed lines of the file:
@@
 Wire Wire Line
 	9650 4300 10600 4300
+$Comp
+L Device:R_Small R?
+U 1 1 5F4B2382
+P 9550 4450
+AR Path="/5F4B2382" Ref="R?"  Part="1"
+AR Path="/5F3EF3FF/5F4B2382" Ref="R235"  Part="1"
+F 0 "R235" V 9500 4300 50  0000 C CNN
+F 1 "R_Small" V 9500 4700 50  0000 C CNN
+F 2 "Resistor_SMD:R_0402_1005Metric" H 9550 4450 50  0001 C CNN
+F 3 "~" H 9550 4450 50  0001 C CNN
+	1    9550 4450
+	0    1    1    0
+$EndComp
+$Comp
+L Device:R_Small R?
+U 1 1 5F4B2626
+P 9550 4550
+AR Path="/5F4B2626" Ref="R?"  Part="1"
+AR Path="/5F3EF3FF/5F4B2626" Ref="R236"  Part="1"
+F 0 "R236" V 9500 4400 50  0000 C CNN
+F 1 "R_Small" V 9500 4800 50  0000 C CNN
+F 2 "Resistor_SMD:R_0402_1005Metric" H 9550 4550 50  0001 C CNN
+F 3 "~" H 9550 4550 50  0001 C CNN
+	1    9550 4550
+	0    1    1    0
+$EndComp
 Wire Wire Line
-	9000 4450 10600 4450
+	9000 4450 9450 4450
 Wire Wire Line
-	9000 4550 10600 4550
+	9450 4550 9000 4550
+Wire Wire Line
+	10600 4450 9650 4450
+Wire Wire Line
+	9650 4550 10600 4550
 Wire Wire Line
 	9000 4650 10600 4650
+$Comp
+L power:GND #PWR0237
+U 1 1 5F96E680
+P 10250 1400
+F 0 "#PWR0237" H 10250 1150 50  0001 C CNN
+F 1 "GND" H 10255 1227 50  0000 C CNN
+F 2 "" H 10250 1400 50  0001 C CNN
+F 3 "" H 10250 1400 50  0001 C CNN
+	1    10250 1400
+	1    0    0    -1
+$EndComp
+$Comp
+L power:GNDD #PWR?
+U 1 1 5F96ED0A
+P 9950 1400
+AR Path="/5F96ED0A" Ref="#PWR?"  Part="1"
+AR Path="/5F3EF3FF/5F96ED0A" Ref="#PWR0235"  Part="1"
+F 0 "#PWR0235" H 9950 1150 50  0001 C CNN
+F 1 "GNDD" H 9954 1245 50  0000 C CNN
+F 2 "" H 9950 1400 50  0001 C CNN
+F 3 "" H 9950 1400 50  0001 C CNN
+	1    9950 1400
+	1    0    0    -1
+$EndComp
+Wire Wire Line
+	9950 1400 10100 1400
+$Comp
+L power:GNDA #PWR?
+U 1 1 5F981646
+P 10100 1600
+AR Path="/5F981646" Ref="#PWR?"  Part="1"
+AR Path="/5F3EF3FF/5F981646" Ref="#PWR0236"  Part="1"
+F 0 "#PWR0236" H 10100 1350 50  0001 C CNN
+F 1 "GNDA" V 10100 1350 50  0000 C CNN
+F 2 "" H 10100 1600 50  0001 C CNN
+F 3 "" H 10100 1600 50  0001 C CNN
+	1    10100 1600
+	1    0    0    -1
+$EndComp
+Wire Wire Line
+	10100 1600 10100 1400
+Connection ~ 10100 1400
+Wire Wire Line
+	10100 1400 10250 1400
+$Comp
+L power:PWR_FLAG #FLG04
+U 1 1 5FA30974
+P 10100 1250
+F 0 "#FLG04" H 10100 1325 50  0001 C CNN
+F 1 "PWR_FLAG" H 10100 1423 50  0000 C CNN
+F 2 "" H 10100 1250 50  0001 C CNN
+F 3 "~" H 10100 1250 50  0001 C CNN
+	1    10100 1250
+	1    0    0    -1
+$EndComp
+Wire Wire Line
+	10100 1250 10100 1400
 $EndSCHEMATC
