File: Schematic/Prosthetic_ARM_DAQ.kicad_pcb (KiCad board)
At the start: 2 copper layers, 157 x 63 mm, 527 parts, among them IC1 ADS1299-4PAGR, IC10 AD8476ACPZ-WP, IC11 ADA4075-2ARZ, IC12 ADA4075-2ARZ, IC13 AD8476ACPZ-WP, IC14 ADA4075-2ARZ, IC15 ADA4075-2ARZ, IC16 AD8476ACPZ-WP, IC17 NJM2068M, IC18 NJM2068M, IC19 AD8476ACPZ-WP, IC2 ADA4075-2ARZ, IC20 ADA4075-2ARZ, IC21 ADA4075-2ARZ, IC22 AD8476ACPZ-WP, IC23 ADA4075-2ARZ, IC24 ADA4075-2ARZ, IC25 AD8476ACPZ-WP, IC3 ADA4075-2ARZ, IC4 AD8476ACPZ-WP, IC5 ADA4075-2ARZ, IC6 ADA4075-2ARZ, IC7 AD8476ACPZ-WP, IC8 ADA4075-2ARZ, IC9 ADA4075-2ARZ, J1 USB4085-GF-A_REVA, J10 Conn_01x03, J2 Conn_01x05, J3 Conn_01x03, J4 Conn_01x03, J5 Conn_01x03, J6 Conn_01x03, J7 Conn_01x03, J8 Conn_01x03, J9 Conn_01x03, U1 STM32F411CEUx

Commit message: Add files via upload
Parts:
- removed the REF** at (92.0, 113.0)
- removed the REF** at (92.0, 184.0)
- added ?: , , F.Cu at (95.3, 100.6)
- added ?: , , F.Cu at (117.3, 11.3)
- added C256: 1N, Capacitor_SMD:C_0402_1005Metric, F.Cu at (154.9, 119.7)
- added C257: 1N, Capacitor_SMD:C_0402_1005Metric, F.Cu at (154.7, 125.0)
- added C258: 100U, Capacitor_SMD:C_0402_1005Metric, B.Cu at (163.0, 112.0)
- added C259: 100U, Capacitor_SMD:C_0402_1005Metric, B.Cu at (155.8, 112.0)
- added C260: 100U, Capacitor_SMD:C_0402_1005Metric, B.Cu at (151.6, 103.7)
- added C261: 100U, Capacitor_SMD:C_0402_1005Metric, B.Cu at (157.7, 100.6)
- added C262: 100U, Capacitor_SMD:C_0402_1005Metric, B.Cu at (160.1, 105.7)
- added C263: 100U, Capacitor_SMD:C_0402_1005Metric, B.Cu at (163.8, 104.0)
- added C264: 1N, Capacitor_SMD:C_0402_1005Metric, F.Cu at (165.8, 130.8)
- added D1: LED, LED_SMD:LED_0805_2012Metric_Pad1.15x1.40mm_HandSolder, F.Cu at (176.2, 130.2)
- added D2: LED, LED_SMD:LED_0805_2012Metric_Pad1.15x1.40mm_HandSolder, F.Cu at (176.2, 133.2)
- added D3: LED, LED_SMD:LED_0805_2012Metric_Pad1.15x1.40mm_HandSolder, F.Cu at (176.2, 136.2)
- added D4: LED, LED_SMD:LED_0805_2012Metric_Pad1.15x1.40mm_HandSolder, F.Cu at (176.2, 139.2)
- added D5: LED, LED_SMD:LED_0805_2012Metric_Pad1.15x1.40mm_HandSolder, F.Cu at (176.2, 142.2)
- added D6: LED, LED_SMD:LED_0805_2012Metric_Pad1.15x1.40mm_HandSolder, F.Cu at (176.2, 145.2)
- added D7: D_Small, Diode_SMD:D_0603_1608Metric_Pad1.05x0.95mm_HandSolder, F.Cu at (172.8, 101.1)
- added D8: D_Small, Diode_SMD:D_0603_1608Metric_Pad1.05x0.95mm_HandSolder, B.Cu at (177.4, 121.4)
- added D9: D_Small, Diode_SMD:D_0603_1608Metric_Pad1.05x0.95mm_HandSolder, B.Cu at (160.0, 102.6)
- added G***: LOGO, ASSETS:Company_Logo1, F.Cu at (158.0, 139.0)
- added IC26: LM2611AMF, ASSETS:SOT95P280X145-5N, B.Cu at (154.6, 103.7)
- added J11: Conn_01x04, Connector_JST:JST_PH_B4B-PH-SM4-TB_1x04-1MP_P2.00mm_Vertical, F.Cu at (162.5, 97.9)
- added L1: L_Small, Inductor_SMD:L_0603_1608Metric_Pad1.05x0.95mm_HandSolder, B.Cu at (154.7, 100.6)
- added L2: L_Small, Inductor_SMD:L_0603_1608Metric_Pad1.05x0.95mm_HandSolder, B.Cu at (162.9, 100.6)
- added R235: R_Small, Resistor_SMD:R_0402_1005Metric, F.Cu at (145.6, 128.5)
- added R236: R_Small, Resistor_SMD:R_0402_1005Metric, F.Cu at (145.6, 130.0)
- added R237: R_Small, Resistor_SMD:R_0402_1005Metric, F.Cu at (171.2, 130.2)
- added R238: R_Small, Resistor_SMD:R_0402_1005Metric, F.Cu at (171.2, 133.2)
- added R239: R_Small, Resistor_SMD:R_0402_1005Metric, F.Cu at (171.2, 136.2)
- added R240: R_Small, Resistor_SMD:R_0402_1005Metric, F.Cu at (171.2, 139.2)
- added R241: R_Small, Resistor_SMD:R_0402_1005Metric, F.Cu at (171.2, 142.2)
- added R242: R_Small, Resistor_SMD:R_0402_1005Metric, F.Cu at (171.2, 145.2)
- added R243: R_Small, Resistor_SMD:R_0402_1005Metric, B.Cu at (166.2, 103.3)
- added R244: R_Small, Resistor_SMD:R_0402_1005Metric, B.Cu at (166.2, 105.8)
- added R245: R_Small, Resistor_SMD:R_0402_1005Metric, B.Cu at (157.8, 103.7)
- added R246: R_Small, Resistor_SMD:R_0402_1005Metric, B.Cu at (157.8, 105.8)
- added REF**: MountingHole_2.5mm_Pad_Via, MountingHole:MountingHole_2.5mm_Pad_Via, F.Cu at (135.6, 109.1)
- added REF**: MountingHole_2.5mm_Pad_Via, MountingHole:MountingHole_2.5mm_Pad_Via, F.Cu at (135.6, 137.9)
- added REF**: 0.5mm-NPTH-Drill, ASSETS:0.5mm-NPTH-Drill, B.Cu at (35.2, 93.6)
- added REF**: 0.5mm-NPTH-Drill, ASSETS:0.5mm-NPTH-Drill, F.Cu at (35.2, 153.4)
- added REF**: MountingHole_2.5mm_Pad_Via, MountingHole:MountingHole_2.5mm_Pad_Via, F.Cu at (20.0, 96.0)
- added REF**: MountingHole_2.5mm_Pad_Via, MountingHole:MountingHole_2.5mm_Pad_Via, F.Cu at (20.0, 151.0)
- added REF**: MountingHole_2.5mm_Pad_Via, MountingHole:MountingHole_2.5mm_Pad_Via, F.Cu at (176.0, 151.0)
- added REF**: MountingHole_2.5mm_Pad_Via, MountingHole:MountingHole_2.5mm_Pad_Via, F.Cu at (176.0, 96.0)
- added U2: AP2127N-3.3, Package_TO_SOT_SMD:SOT-23, B.Cu at (159.4, 111.9)
- added Y1: Crystal_GND23, Crystal:Crystal_SMD_TXC_7M-4Pin_3.2x2.5mm, F.Cu at (154.9, 122.4)
- C100, C101, C102, C103, C104, C105, C106, C107, C108, C109, C110, C111, C112, C113, C114, C115, C228, C229, C230, C231, C232, C233, C234, C235, C236, C237, C238, C239, C240, C241, C242, C243, C244, C245, C246, C247, C248, C249, C250, C251, C252, C253, C254, C255, C32, C33, C34, C35, C36, C37, C38, C39, C40, C41, C42, C43, C44, C45, C46, C47, C48, C49, C50, C51, C52, C53, C54, C55, C56, C57, C58, C59, C60, C61, C62, C63, C64, C65, C66, C67, C68, C69, C70, C71, C72, C73, C74, C75, C76, C77, C78, C79, C80, C81, C82, C83, C84, C85, C86, C87, C88, C89, C90, C91, C92, C93, C94, C95, C96, C97, C98, C99, IC10, IC2, IC23, IC24, IC25, IC3, IC4, IC5, IC6, IC7, IC8, IC9, J10, J3, J4, J5, R100, R101, R102, R103, R104, R209, R210, R211, R212, R213, R214, R215, R216, R217, R218, R219, R220, R221, R222, R223, R224, R225, R226, R227, R228, R229, R230, R231, R232, R233, R234, R27, R28, R29, R30, R31, R32, R33, R34, R35, R36, R37, R38, R39, R40, R41, R42, R43, R44, R45, R46, R47, R48, R49, R50, R51, R52, R53, R54, R55, R56, R57, R58, R59, R60, R61, R62, R63, R64, R65, R66, R67, R68, R69, R70, R71, R72, R73, R74, R75, R76, R77, R78, R79, R80, R81, R82, R83, R84, R85, R86, R87, R88, R89, R90, R91, R92, R93, R94, R95, R96, R97, R98, R99: moved to B.Cu
- IC17, IC18: value NJM2068M -> ADA4075-2ARZ; footprint ASSETS:SOIC127P680X200-8N -> ASSETS:SOIC127P600X175-8N
- moved J10 255.5 mm to (29.6, 147.0), turned to 270 degrees
- moved R11 254.2 mm to (115.6, 146.0), turned to 180 degrees
- moved R12 252.1 mm to (115.6, 150.0)
- moved C59 250.8 mm to (80.1, 149.1), turned to 270 degrees
- moved C231 250.5 mm to (41.3, 129.3), turned to 180 degrees
- moved J3 249.7 mm to (29.6, 130.7), turned to 270 degrees
- moved C15 246.7 mm to (116.6, 148.0), turned to 270 degrees
- moved C57 246.1 mm to (82.5, 149.1), turned to 270 degrees
- moved R234 245.0 mm to (63.4, 142.2)
- moved C242 244.3 mm to (51.9, 132.5)
- moved C241 243.4 mm to (51.7, 147.2), turned to 0 degrees
- moved R212 243.1 mm to (41.3, 146.1), turned to 90 degrees
- moved IC25 243.1 mm to (63.4, 138.1)
- moved R217 242.0 mm to (51.2, 143.2), turned to 90 degrees
- moved C238 241.9 mm to (51.7, 146.1), turned to 0 degrees
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Connections:
- net STATUS_IND_LED renamed Net-(U1-Pad2)
- C1 pad 1: +3V3 -> Net-(C1-Pad1)
- C19 pad 2: GNDA -> GND
- C20 pad 2: GNDA -> GND
- C21 pad 1: GNDA -> GND
- C22 pad 2: GNDA -> GND
- C23 pad 1: GNDA -> GND
- C24 pad 1: GNDA -> GND
- C25 pad 1: GNDA -> GND
- C26 pad 1: GNDA -> GND
- C27 pad 2: GNDA -> GND
- C28 pad 1: GNDA -> GND
- C29 pad 1: GNDD -> GND
- C30 pad 1: GNDA -> GND
- C31 pad 2: GNDD -> GND
- IC1 pad 20: GNDA -> GND
- IC1 pad 23: GNDA -> GND
- IC1 pad 25: GNDA -> GND
- IC1 pad 32: GNDA -> GND
- IC1 pad 33: GNDD -> GND
- IC1 pad 35: nPWDN -> Net-(IC1-Pad35)
- IC1 pad 36: nRESET -> Net-(IC1-Pad36)
- IC1 pad 41: GNDD -> GND
- IC1 pad 49: GNDD -> GND
- IC1 pad 51: GNDD -> GND
- IC1 pad 53: GNDA -> GND
- IC1 pad 56: GNDA -> GND
- IC1 pad 58: GNDA -> GND
- IC10 pad 17: Net-(IC10-Pad17) -> GND
- IC13 pad 17: Net-(IC13-Pad17) -> GND
- IC16 pad 17: Net-(IC16-Pad17) -> GND
- IC17 pad 5: Net-(C177-Pad1) -> Net-(C178-Pad1)
- IC17 pad 7: /Analog_AFE/sheet5F407F6C/IN1 -> /Analog_AFE/sheet5F407F6C/IN2
- IC18 pad 5: Net-(C178-Pad1) -> Net-(C177-Pad1)
- IC18 pad 7: /Analog_AFE/sheet5F407F6C/IN2 -> /Analog_AFE/sheet5F407F6C/IN1
- IC19 pad 17: Net-(IC19-Pad17) -> GND
- IC22 pad 17: Net-(IC22-Pad17) -> GND
- IC25 pad 17: Net-(IC25-Pad17) -> GND
- IC4 pad 17: Net-(IC4-Pad17) -> GND
- IC7 pad 17: Net-(IC7-Pad17) -> GND
- J1 pad A4: +3V3 -> Net-(D8-Pad2)
- J1 pad A6: DP+ -> DN_P
- J1 pad A7: DN- -> DN_N
- J1 pad A9: +3V3 -> Net-(D8-Pad2)
- J1 pad B4: +3V3 -> Net-(D8-Pad2)
- J1 pad B6: DP+ -> DN_P
- J1 pad B7: DN- -> DN_N
- J1 pad B9: +3V3 -> Net-(D8-Pad2)
- J2 pad 1: +3V3 -> Net-(C1-Pad1)
- J8 pad 1: Net-(IC17-Pad3) -> Net-(IC18-Pad3)
- J8 pad 3: Net-(IC18-Pad3) -> Net-(IC17-Pad3)
- R157 pad 1: Net-(IC17-Pad2) -> Net-(IC18-Pad2)
- R158 pad 1: Net-(IC18-Pad2) -> Net-(IC17-Pad2)
- R159 pad 1: Net-(IC17-Pad1) -> Net-(IC18-Pad1)
- R159 pad 2: Net-(IC17-Pad2) -> Net-(IC18-Pad2)
- R160 pad 1: Net-(IC18-Pad1) -> Net-(IC17-Pad1)
- R160 pad 2: Net-(IC18-Pad2) -> Net-(IC17-Pad2)
- R163 pad 2: Net-(IC17-Pad6) -> Net-(IC18-Pad6)
- R165 pad 2: Net-(IC18-Pad6) -> Net-(IC17-Pad6)
- R167 pad 1: Net-(IC17-Pad6) -> Net-(IC18-Pad6)
- R168 pad 1: Net-(IC18-Pad6) -> Net-(IC17-Pad6)
- R179 pad 2: Net-(IC17-Pad1) -> Net-(IC18-Pad1)
- R180 pad 2: Net-(IC18-Pad1) -> Net-(IC17-Pad1)
- U1 pad 1: VBAT -> +3V3
- U1 pad 12: Net-(U1-Pad12) -> GPIO1
- U1 pad 13: Net-(U1-Pad13) -> START
- U1 pad 18: Net-(U1-Pad18) -> nRESET
- U1 pad 19: Net-(U1-Pad19) -> nPWDN
- U1 pad 22: VCAP1 -> +3V3
- U1 pad 27: Net-(U1-Pad27) -> LED5
- U1 pad 28: Net-(U1-Pad28) -> LED4
- U1 pad 29: Net-(U1-Pad29) -> LED3
- U1 pad 30: Net-(U1-Pad30) -> LED2
- U1 pad 31: Net-(U1-Pad31) -> LED1
- U1 pad 32: Net-(U1-Pad32) -> DN_N
- U1 pad 33: Net-(U1-Pad33) -> DN_P
- U1 pad 38: Net-(U1-Pad38) -> USART_TX
- U1 pad 39: Net-(U1-Pad39) -> USART_RX
- U1 pad 40: Net-(U1-Pad40) -> SLAVE_READY
- U1 pad 42: Net-(U1-Pad42) -> DRDY
- U1 pad 43: Net-(U1-Pad43) -> GPIO4
- U1 pad 44: BOOT0 -> GND
- U1 pad 45: Net-(U1-Pad45) -> GPIO3
- U1 pad 46: Net-(U1-Pad46) -> GPIO2
- U1 pad 7: RESET -> +3V3
Routing:
- net GND: track 0.00 -> 194.0 mm, vias 0 -> 101
- net +3V3: track 18.9 -> 116.5 mm, vias 0 -> 1
- net -3V3: track 20.6 -> 79.9 mm
- net SWO: track 0.00 -> 35.2 mm, vias 0 -> 1
- net /Analog_AFE/sheet5F407F68/IN1: track 0.00 -> 34.2 mm
- net /Analog_AFE/sheet5F407F67/IN1: track 0.00 -> 33.7 mm
- net Net-(C15-Pad2): track 0.00 -> 31.6 mm
- net Net-(C15-Pad1): track 0.00 -> 31.4 mm
- net Net-(C10-Pad1): track 0.00 -> 31.3 mm
- net Net-(C10-Pad2): track 0.00 -> 31.1 mm
- net /Analog_AFE/sheet5F407F6E/IN1: track 2.61 -> 33.4 mm
- net /Analog_AFE/sheet5F407F67/IN2: track 0.00 -> 29.6 mm
- net /Analog_AFE/sheet5F407F68/IN2: track 0.00 -> 28.5 mm
- net DIN: track 0.00 -> 28.1 mm, vias 0 -> 2
- net /Analog_AFE/sheet5F407F6E/IN2: track 2.65 -> 29.1 mm
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- added copper zone on B.Cu, net GND
- added copper zone on F.Cu, net GND
- added copper zone on GND, net GND
Other:
- board size 157 x 63 mm -> 164.4 x 63 mm
- copper layers 2 -> 4
- board text added: "3.3V"
- board text added: "Axion Embedded"
- board text added: "GND"
- board text added: "SLV_READY"
- board text added: "SWCLK"
- board text added: "SWDIO"
- board text added: "SWO"
- board text added: "UART_RX"
- board text added: "UART_TX"
